File: Lab8_Flightboard_Starter.kicad_sch (KiCad schematic)
At the start: 64 parts, among them J1 Motor1, J10 ESC3_GND, J11 ESC4_VBAT, J12 ESC4_GND, J2 Motor2, J3 Motor3, J4 Motor4, J5 ESC1_VBAT, J6 ESC1_GND, J7 ESC2_VBAT, J8 ESC2_GND, J9 ESC3_VBAT, Q1 DMP6023LE-13, U1 Teensy4.0, U2 TPS62933, U4 LP5912-3.3DRV, U5 LP5912-3.3DRV, U6 NRF24L01_Breakout, U9 LSM6DSO32_Adafruit

Commit message: Fixed MCU wiring
Connections:
- net CE: now also U1.11 (9_OUT1C); no longer U1.9 (7_RX2_OUT1A)
- net CS: now also U1.28 (21_A7_RX5_BCLK1); no longer U1.12 (10_CS_MQSR)
- net CSN: now also U1.12 (10_CS_MQSR); no longer U1.11 (9_OUT1C)
- net M1_CMD: now also U1.10 (8_TX2_IN1); no longer U1.6 (4_BCLK2)
- net M2_CMD: now also U1.6 (4_BCLK2); no longer U1.10 (8_TX2_IN1)
- net SCK: now also U1.20 (13_SCK_CRX1_LED); no longer U1.21 (14_A0_TX3_SPDIF_OUT)
- net VBAT_SENSE: now also U1.27 (20_A6_TX5_LRCLK1); no longer U1.22 (15_A1_RX3_SPDIF_IN)
- net ADC3 renamed ADC6

Commit message: Fixed wire warning
Connections:
- net ADC6 renamed ADC3
Changed lines of the file:
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@@
-	(wire
-		(pts
-			(xy 147.855 242.1017) (xy 139.7 242.57)
-		)
-		(stroke
-			(width 0)
-			(type default)
-		)
-	)
 	(wire
 		(pts
@@
 		)
 	)
-	(label "ADC6"
+	(label "ADC3"
 		(at 58.42 191.77 180)
 		(effects
@@
 		)
 	)
-	(label "ADC6"
-		(at 147.855 242.1017 180)
-		(effects
-			(font
+	(label "ADC3"
+		(at 139.7 242.57 180)
+		(effects
+			(font

Commit message: Remade the power plane + updates
Connections:
- net SYS_VIN: now also R4.2
- net VBAT: no longer R4.2
Changed lines of the file:
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@@
 		)
 	)
-	(label "VBAT"
+	(label "SYS_VIN"
 		(at 252.73 39.37 180)
 		(effects

Commit message: Improved the design
Parts:
- R10, R12, R6, R8: value 47 -> 100k
- R11, R13, R7, R9: value 100k -> 47
Changed lines of the file:
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@@
 			)
 		)
-		(property "Value" "100k"
+		(property "Value" "47"
 			(at 299.72 185.928 90)
 			(show_name no)
@@
 			)
 		)
-		(property "Value" "47"
+		(property "Value" "100k"
 			(at 292.1 186.182 90)
 			(show_name no)
@@
 			)
 		)
-		(property "Value" "100k"
+		(property "Value" "47"
 			(at 299.466 195.9628 90)
 			(show_name no)
@@
 			)
 		)
-		(property "Value" "100k"
+		(property "Value" "47"
 			(at 299.72 175.768 90)
 			(show_name no)
@@
 			)
 		)
-		(property "Value" "47"
+		(property "Value" "100k"
 			(at 291.7172 196.342 90)
 			(show_name no)
@@
 			)
 		)
-		(property "Value" "100k"
+		(property "Value" "47"
 			(at 299.72 165.354 90)
 			(show_name no)
@@
 			)
 		)
-		(property "Value" "47"
+		(property "Value" "100k"
 			(at 291.846 176.022 90)
 			(show_name no)
@@
 			)
 		)
-		(property "Value" "47"
+		(property "Value" "100k"
 			(at 292.1 165.1 90)
 			(show_name no)
